Commit message: Inverse Kinematics Example 1

File: asset/URDF_ALLEX_RightArm/urdf/URDF_ALLEX_RightArm.urdf (robot description, URDF)
Before this commit: robot URDF_ALLEX_RightArm, 9 links, 8 joints
Joints:
- joint EP: limit lower=-1 upper=1 effort=150 velocity=10 -> lower=-2.87979 upper=0.0872665 effort=150 velocity=10
- joint EY: limit lower=-1 upper=1 effort=150 velocity=10 -> lower=-0.610865 upper=4.79966 effort=150 velocity=10
- joint SP: limit lower=-1 upper=1 effort=200 velocity=10 -> lower=-3.31613 upper=1.74533 effort=200 velocity=10
- joint SR: limit lower=-1 upper=1 effort=180 velocity=10 -> lower=-3.75246 upper=0.0872665 effort=180 velocity=10
- joint SY: limit lower=-1 upper=1 effort=150 velocity=10 -> lower=-1.74533 upper=3.31613 effort=150 velocity=10
- joint WP: limit lower=-1 upper=1 effort=120 velocity=10 -> lower=-1.39626 upper=1.39626 effort=120 velocity=10
- joint WR: limit lower=-1 upper=1 effort=120 velocity=10 -> lower=-0.872665 upper=0.872665 effort=120 velocity=10
